Commit message: update lingao_description

File: lingao_description/urdf/LA_4WD_LingFeng.urdf (robot description, URDF)
Before this commit: robot lingao_description, 5 links, 4 joints
Links:
- link base_link: mass 0.43668 -> None
- link wheel_la_link: mass 0.72164 -> None
- link wheel_lb_link: mass 0.72164 -> None
- link wheel_ra_link: mass 0.72164 -> None
- link wheel_rb_link: mass 0 -> None
