Commit message: fix UnicodeEncodeError

File: lingao_description/urdf/MiniUGV_10A.xacro (robot description, xacro)
@@ -7,5 +7,5 @@
     <xacro:property name="base_width" value="0.345"/>
     <xacro:property name="base_height" value="0.184"/>
-    <xacro:property name="earth_space" value="0.055" /> <!-- 离地间距 -->
+    <xacro:property name="earth_space" value="0.055" />
     <!-- Base link -->
     <link name="base_link">

Commit message: update lingao xarco

File: lingao_description/urdf/MiniUGV_10A.xacro (robot description, xacro)
@@ -13,5 +13,5 @@
         <origin xyz="0 0 0" rpy="0 0 0" />
         <geometry>
-            <mesh filename="file://$(find lingao_description)/meshes/LA_MiniUGV_10A/mobile_base.stl" scale="1 1 1"/>
+            <mesh filename="package://lingao_description/meshes/LA_MiniUGV_10A/mobile_base.stl" scale="1 1 1"/>
         </geometry>
         <material name="yellow">
@@ -44,5 +44,5 @@
                 <origin xyz="0 0 0" rpy="0 0 0" />
                 <geometry>
-                    <mesh filename="file://$(find lingao_description)/meshes/LA_MiniUGV_10A/mobile_whell.stl" />
+                    <mesh filename="package://lingao_description/meshes/LA_MiniUGV_10A/mobile_whell.stl" />
                 </geometry>
                 <material name="Poppy">
